File: eagleclone/spec/OpAmp-breakout-ABC.brd (EAGLE design)
At the start: 12.7 x 24.1 mm, 19 parts, among them IC1-ABC LMV358

Commit message: added some more of the common power names so they don't get translated
Connections:
- net VCC-ABC renamed VCC
Changed lines of the file:
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@@
 <wire x1="9.144" y1="11.811" x2="10.16" y2="10.795" width="0.254" layer="1"/>
 </signal>
-<signal name="VCC-ABC">
+<signal name="VCC">
 <contactref element="JP1-ABC" pad="1"/>
 <contactref element="C2-ABC" pad="1"/>
