File: eagleclone/spec/OpAmp-breakout-ABC.sch (EAGLE design)
At the start: 17 parts, among them IC1-ABC LMV358

Commit message: added some more of the common power names so they don't get translated
Connections:
- net VCC-ABC renamed VCC
Changed lines of the file:
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@@
 </segment>
 </net>
-<net name="VCC-ABC" class="0">
+<net name="VCC" class="0">
 <segment>
 <wire x1="109.22" y1="101.6" x2="106.68" y2="101.6" width="0.1524" layer="91"/>
